Commit message: modified URDF of 1d hopper for import

File: demos/hopper_1d.urdf (robot description, URDF)
Before this commit: robot hopper, 5 links, 4 joints
Links:
- link contact: geometry collision sphere radius=0.025; visual mesh filename=package://quadruped/meshes/sphere.obj scale=0.025 0.025 0.025
- link lower_leg: geometry collision cylinder length=0.16 radius=0.025; visual mesh filename=package://quadruped/meshes/cylinder.obj scale=0.025 0.025 0.16
- link shank: geometry collision cylinder length=0.16 radius=0.025; visual mesh filename=package://quadruped/meshes/cylinder.obj scale=0.025 0.025 0.16

Commit message: started with the impedance controller for Teststand and Quadruped

File: demos/hopper_1d.urdf (robot description, URDF)
Before this commit: robot hopper, 5 links, 4 joints
Links:
- link contact: geometry collision sphere radius=0.025
- link lower_leg: geometry collision cylinder length=0.16 radius=0.025
- link shank: geometry collision cylinder length=0.16 radius=0.025
